File: eCog_UART_Template.brd (EAGLE design)
At the start: 48 x 28 mm, 1 part

Commit message: V1.1
Parts:
- ECOG: value ECOG_BUSES_ROWECOG_BUSES_SMD -> ECOG_GENERAL_ROWECOG_GENERAL_SMD; device eCogs:ECOG_BUSES_SMD -> eCogs:ECOG_GENERAL_SMD
Connections:
- new net RX: ECOG.2
- new net TX: ECOG.1
Other:
- board text added: "P1<>"
- board text added: "P2<>"
- board text added: "P3<>"
- board text added: "P4<>"
- board text added: "P6<>"
- board text added: "P7<>"
- board text added: "P8<>"
- board text removed: "I2C-SCL"
- board text removed: "I2C-SDA"
- board text removed: "RESET"
- board text removed: "SPI-CS>"
- board text removed: "SPI-MOSI<"
- board text removed: "SPI-MOSI>"
- board text removed: "SPI-SCK>"
Changed lines of the file:
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@@
 <text x="28.702" y="3.429" size="1.016" layer="21" font="vector">Project Name</text>
 <text x="28.702" y="4.699" size="1.016" layer="21" font="vector">eCogs</text>
-<text x="1.095" y="26.162" size="1.016" layer="21" font="vector">SPI-MOSI&lt;</text>
-<text x="1.095" y="23.622" size="1.016" layer="21" font="vector">SPI-MOSI&gt;</text>
-<text x="1.095" y="21.082" size="1.016" layer="21" font="vector">SPI-SCK&gt;</text>
-<text x="1.095" y="18.542" size="1.016" layer="21" font="vector">SPI-CS&gt;</text>
-<text x="1.095" y="16.002" size="1.016" layer="21" font="vector">P5&lt;&gt;</text>
-<text x="1.095" y="13.462" size="1.016" layer="21" font="vector">I2C-SDA</text>
-<text x="1.095" y="10.922" size="1.016" layer="21" font="vector">I2C-SCL</text>
-<text x="1.095" y="3.302" size="1.016" layer="21" font="vector">RESET</text>
+<text x="1.175" y="26.162" size="1.016" layer="21" font="vector">P1&lt;&gt;</text>
+<text x="1.175" y="23.622" size="1.016" layer="21" font="vector">P2&lt;&gt;</text>
+<text x="1.175" y="21.082" size="1.016" layer="21" font="vector">P3&lt;&gt;</text>
+<text x="1.175" y="18.542" size="1.016" layer="21" font="vector">P4&lt;&gt;</text>
+<text x="1.175" y="16.002" size="1.016" layer="21" font="vector">P5&lt;&gt;</text>
+<text x="1.175" y="13.462" size="1.016" layer="21" font="vector">P6&lt;&gt;</text>
+<text x="1.175" y="10.922" size="1.016" layer="21" font="vector">P7&lt;&gt;</text>
+<text x="1.175" y="3.302" size="1.016" layer="21" font="vector">P8&lt;&gt;</text>
 <text x="33.782" y="17.526" size="0.6096" layer="21" font="vector">Copyright 2016</text>
 <text x="32.512" y="16.637" size="0.6096" layer="21" font="vector">Gadget Factory, LLC</text>
-<text x="1.095" y="8.382" size="1.016" layer="21" font="vector">5V</text>
-<text x="1.095" y="5.842" size="1.016" layer="21" font="vector">3.3V</text>
-<text x="1.095" y="0.762" size="1.016" layer="21" font="vector">GND</text>
+<text x="1.175" y="8.382" size="1.016" layer="21" font="vector">5V</text>
+<text x="1.175" y="5.842" size="1.016" layer="21" font="vector">3.3V</text>
+<text x="1.175" y="0.762" size="1.016" layer="21" font="vector">GND</text>
 </plain>
 <attributes>
@@
 </autorouter>
 <elements>
-<element name="ECOG" library="eCogs" package="ECOG_BUSES_SMD" value="ECOG_BUSES_ROWECOG_BUSES_SMD" x="0" y="0" smashed="yes"/>
+<element name="ECOG" library="eCogs" package="ECOG_GENERAL_SMD" value="ECOG_GENERAL_ROWECOG_GENERAL_SMD" x="0" y="0" smashed="yes"/>
 </elements>
 <signals>
@@
 <contactref element="ECOG" pad="GND"/>
 </signal>
+<signal name="TX">
+<contactref element="ECOG" pad="1"/>
+</signal>
+<signal name="RX">
+<contactref element="ECOG" pad="2"/>
+</signal>
 <signal name="3V3">
 <contactref element="ECOG" pad="3V3"/>
@@
 <vertex x="0" y="0"/>
 </polygon>
-<wire x1="7.9002" y1="6.4054" x2="10.1046" y2="6.4054" width="0.6096" layer="16"/>
-<wire x1="10.1046" y1="6.4054" x2="10.16" y2="6.35" width="0.6096" layer="16"/>
-<via x="10.16" y="6.35" extent="1-16" drill="0.381"/>
-<wire x1="10.16" y1="6.35" x2="10.16" y2="7.62" width="0.6096" layer="1"/>
+<wire x1="5.3494" y1="6.38" x2="7.59" y2="6.38" width="0.6096" layer="16"/>
+<wire x1="7.59" y1="6.38" x2="7.62" y2="6.35" width="0.6096" layer="16"/>
+<via x="7.62" y="6.35" extent="1-16" drill="0.381"/>
+<wire x1="7.62" y1="6.35" x2="7.62" y2="7.62" width="0.6096" layer="1"/>
 </signal>
 </signals>

Commit message: Latest updated to V1.4
Parts:
- added U$1: (no value), GadgetFactory:GADGETBOX_TEXT
- added U$2, U$3: (no value), eCogs:LEGEND_DIO
- added U$4, U$5, U$6: (no value), eCogs:LEGEND_PWM
- added U$7, U$8, U$9: (no value), eCogs:LEGEND_ANALOG
Connections:
- net RX: now also ECOG.G1; no longer ECOG.2
- net TX: now also ECOG.G0; no longer ECOG.1
Routing:
- net 3V3: track 3.55 -> 2.56 mm
Other:
- outline, holes or cut-outs redrawn
- board text added: "G0<>"
- board text added: "G1<>"
- board text added: "G2<>"
- board text added: "G3<>"
- board text added: "G4<>"
- board text added: "G5<>"
- board text added: "G6<>"
- board text added: "G7<>"
- board text removed: "5V"
- board text removed: "P1<>"
- board text removed: "P2<>"
- board text removed: "P3<>"
- board text removed: "P4<>"
- board text removed: "P5<>"
- board text removed: "P6<>"
- board text removed: "P7<>"
- board text removed: "P8<>"
