File: Gadget-Box-mini-pro.sch (EAGLE design)
At the start: 21 parts, among them U1 MCP73831T-2ACI/OT, U2 AP2112-3.3, X1 USB-MICROB, X100 JSTPH

Commit message: GB Mini Pro V1.2
Parts:
- removed X1: USB-MICROB, SparkFun:USB-MICROB
- added JP1: (no value), SparkFun:M02-JST-2-PTH-NO_SILK
- added JP2, JP3: (no value), SparkFun:M02POGO_PIN_HOLES_ONLY
- added PWR: (no value), adafruit:USBMINIB
- added R4, R7: 10K, GadgetFactory:R0805
Connections:
- net 3V3: now also R4A.2, R7A.2, U$1.VCC1
- net 5V0: now also PWR.VBUS; no longer X1.VBUS
- net D0/RX: now also U$1.TX0-1
- net D1/TX: now also U$1.RX1-1
- net GND: now also JP1.1, PWR.GND, U$1.GND3, U$1.GND4; no longer X1.GND
- net I2C-SCL: now also R7A.1
- net I2C-SDA: now also R4A.1
- net RESET: now also AH.RESET@1, AL.RESET@1, BH.RESET@1, BL.RESET@1, U$1.DTR
- net VBAT: now also JP1.2

Commit message: Fixed the backwards rx and tx lines.
Connections:
- net D0/RX: now also U$1.RX1, U$1.RX1-1; no longer U$1.TX0, U$1.TX0-1
- net D1/TX: now also U$1.TX0, U$1.TX0-1; no longer U$1.RX1, U$1.RX1-1
Changed lines of the file:
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@@
-</segment>
-<segment>
-<wire x1="114.3" y1="152.4" x2="104.14" y2="152.4" width="0.2032" layer="91"/>
-<label x="104.14" y="152.4" size="1.778" layer="95"/>
-<pinref part="U$1" gate="G$1" pin="TX0"/>
 </segment>
 <segment>
@@
 </segment>
 <segment>
-<pinref part="U$1" gate="G$1" pin="TX0-1"/>
-<wire x1="137.16" y1="167.64" x2="137.16" y2="172.72" width="0.2032" layer="91"/>
-<label x="137.16" y="167.64" size="1.778" layer="95" rot="R90"/>
+<wire x1="114.3" y1="149.86" x2="104.14" y2="149.86" width="0.2032" layer="91"/>
+<label x="104.14" y="149.86" size="1.778" layer="95"/>
+<pinref part="U$1" gate="G$1" pin="RX1"/>
+</segment>
+<segment>
+<pinref part="U$1" gate="G$1" pin="RX1-1"/>
+<wire x1="134.62" y1="167.64" x2="134.62" y2="172.72" width="0.2032" layer="91"/>
+<label x="134.62" y="167.64" size="1.778" layer="95" rot="R90"/>
 </segment>
 </net>
@@
 </segment>
 <segment>
-<wire x1="114.3" y1="149.86" x2="104.14" y2="149.86" width="0.2032" layer="91"/>
-<label x="104.14" y="149.86" size="1.778" layer="95"/>
-<pinref part="U$1" gate="G$1" pin="RX1"/>
+<wire x1="114.3" y1="152.4" x2="104.14" y2="152.4" width="0.2032" layer="91"/>
+<label x="104.14" y="152.4" size="1.778" layer="95"/>
+<pinref part="U$1" gate="G$1" pin="TX0"/>
 </segment>
 <segment>
-<pinref part="U$1" gate="G$1" pin="RX1-1"/>
-<wire x1="134.62" y1="167.64" x2="134.62" y2="172.72" width="0.2032" layer="91"/>
-<label x="134.62" y="167.64" size="1.778" layer="95" rot="R90"/>
+<pinref part="U$1" gate="G$1" pin="TX0-1"/>
+<wire x1="137.16" y1="167.64" x2="137.16" y2="172.72" width="0.2032" layer="91"/>
+<label x="137.16" y="167.64" size="1.778" layer="95" rot="R90"/>
 </segment>
 </net>

Commit message: Update Silkscreen
Connections:
- net D0/RX: no longer AL.SPI-CS@B3
- net D7/A3: now also BH.SPI-CS@B3
- net SPI-CS1: now also AL.SPI-CS@B3; no longer BH.SPI-CS@B3
Changed lines of the file:
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@@
 <grid distance="0.1" unitdist="inch" unit="inch" style="lines" multiple="1" display="no" altdistance="0.01" altunitdist="inch" altunit="inch"/>
 <layers>
-<layer number="1" name="Top" color="4" fill="1" visible="yes" active="no"/>
-<layer number="2" name="Route2" color="1" fill="3" visible="yes" active="no"/>
-<layer number="3" name="Route3" color="4" fill="3" visible="yes" active="no"/>
-<layer number="14" name="Route14" color="1" fill="6" visible="yes" active="no"/>
-<layer number="15" name="Route15" color="4" fill="6" visible="yes" active="no"/>
-<layer number="16" name="Bottom" color="1" fill="1" visible="yes" active="no"/>
-<layer number="17" name="Pads" color="2" fill="1" visible="yes" active="no"/>
-<layer number="18" name="Vias" color="2" fill="1" visible="yes" active="no"/>
-<layer number="19" name="Unrouted" color="6" fill="1" visible="yes" active="no"/>
-<layer number="20" name="Dimension" color="15" fill="1" visible="yes" active="no"/>
-<layer number="21" name="tPlace" color="16" fill="1" visible="yes" active="no"/>
-<layer number="22" name="bPlace" color="14" fill="1" visible="yes" active="no"/>
-<layer number="23" name="tOrigins" color="15" fill="1" visible="yes" active="no"/>
-<layer number="24" name="bOrigins" color="15" fill="1" visible="yes" active="no"/>
-<layer number="25" name="tNames" color="16" fill="1" visible="yes" active="no"/>
-<layer number="26" name="bNames" color="7" fill="1" visible="yes" active="no"/>
-<layer number="27" name="tValues" color="7" fill="1" visible="yes" active="no"/>
-<layer number="28" name="bValues" color="7" fill="1" visible="yes" active="no"/>
+<layer number="1" name="Top" color="4" fill="1" visible="no" active="no"/>
+<layer number="2" name="Route2" color="1" fill="3" visible="no" active="no"/>
+<layer number="3" name="Route3" color="4" fill="3" visible="no" active="no"/>
+<layer number="14" name="Route14" color="1" fill="6" visible="no" active="no"/>
+<layer number="15" name="Route15" color="4" fill="6" visible="no" active="no"/>
+<layer number="16" name="Bottom" color="1" fill="1" visible="no" active="no"/>
+<layer number="17" name="Pads" color="2" fill="1" visible="no" active="no"/>
+<layer number="18" name="Vias" color="2" fill="1" visible="no" active="no"/>
+<layer number="19" name="Unrouted" color="6" fill="1" visible="no" active="no"/>
+<layer number="20" name="Dimension" color="15" fill="1" visible="no" active="no"/>
+<layer number="21" name="tPlace" color="16" fill="1" visible="no" active="no"/>
+<layer number="22" name="bPlace" color="14" fill="1" visible="no" active="no"/>
+<layer number="23" name="tOrigins" color="15" fill="1" visible="no" active="no"/>
+<layer number="24" name="bOrigins" color="15" fill="1" visible="no" active="no"/>
+<layer number="25" name="tNames" color="16" fill="1" visible="no" active="no"/>
+<layer number="26" name="bNames" color="7" fill="1" visible="no" active="no"/>
+<layer number="27" name="tValues" color="7" fill="1" visible="no" active="no"/>
+<layer number="28" name="bValues" color="7" fill="1" visible="no" active="no"/>
 <layer number="29" name="tStop" color="7" fill="3" visible="no" active="no"/>
 <layer number="30" name="bStop" color="7" fill="6" visible="no" active="no"/>
@@
 <layer number="35" name="tGlue" color="7" fill="4" visible="no" active="no"/>
 <layer number="36" name="bGlue" color="7" fill="5" visible="no" active="no"/>
-<layer number="37" name="tTest" color="7" fill="1" visible="yes" active="no"/>
-<layer number="38" name="bTest" color="7" fill="1" visible="yes" active="no"/>
+<layer number="37" name="tTest" color="7" fill="1" visible="no" active="no"/>
+<layer number="38" name="bTest" color="7" fill="1" visible="no" active="no"/>
 <layer number="39" name="tKeepout" color="4" fill="11" visible="no" active="no"/>
 <layer number="40" name="bKeepout" color="1" fill="11" visible="no" active="no"/>
@@
 <layer number="44" name="Drills" color="7" fill="1" visible="no" active="no"/>
 <layer number="45" name="Holes" color="7" fill="1" visible="no" active="no"/>
-<layer number="46" name="Milling" color="3" fill="1" visible="yes" active="no"/>
-<layer number="47" name="Measures" color="7" fill="1" visible="yes" active="no"/>
-<layer number="48" name="Document" color="7" fill="1" visible="yes" active="no"/>
-<layer number="49" name="Reference" color="7" fill="1" visible="yes" active="no"/>
-<layer number="50" name="dxf" color="7" fill="1" visible="yes" active="no"/>
-<layer number="51" name="tDocu" color="6" fill="1" visible="yes" active="no"/>
-<layer number="52" name="bDocu" color="7" fill="1" visible="yes" active="no"/>
-<layer number="53" name="tGND_GNDA" color="7" fill="1" visible="yes" active="no"/>
-<layer number="54" name="bGND_GNDA" color="7" fill="1" visible="yes" active="no"/>
-<layer number="56" name="wert" color="7" fill="1" visible="yes" active="no"/>
-<layer number="57" name="tCAD" color="7" fill="1" visible="yes" active="no"/>
-<layer number="59" name="tCarbon" color="7" fill="1" visible="yes" active="no"/>
-<layer number="60" name="bCarbon" color="7" fill="1" visible="yes" active="no"/>
+<layer number="46" name="Milling" color="3" fill="1" visible="no" active="no"/>
+<layer number="47" name="Measures" color="7" fill="1" visible="no" active="no"/>
+<layer number="48" name="Document" color="7" fill="1" visible="no" active="no"/>
+<layer number="49" name="Reference" color="7" fill="1" visible="no" active="no"/>
+<layer number="50" name="dxf" color="7" fill="1" visible="no" active="no"/>
+<layer number="51" name="tDocu" color="6" fill="1" visible="no" active="no"/>
+<layer number="52" name="bDocu" color="7" fill="1" visible="no" active="no"/>
+<layer number="53" name="tGND_GNDA" color="7" fill="1" visible="no" active="no"/>
+<layer number="54" name="bGND_GNDA" color="7" fill="1" visible="no" active="no"/>
+<layer number="56" name="wert" color="7" fill="1" visible="no" active="no"/>
+<layer number="57" name="tCAD" color="7" fill="1" visible="no" active="no"/>
+<layer number="59" name="tCarbon" color="7" fill="1" visible="no" active="no"/>
+<layer number="60" name="bCarbon" color="7" fill="1" visible="no" active="no"/>
 <layer number="90" name="Modules" color="7" fill="1" visible="yes" active="yes"/>
 <layer number="91" name="Nets" color="2" fill="1" visible="yes" active="yes"/>
@@
 </segment>
 <segment>
-<label x="170.18" y="93.98" size="1.778" layer="95"/>
-<pinref part="AL" gate="ECOG$1" pin="SPI-CS@B3"/>
-<wire x1="182.88" y1="93.98" x2="157.48" y2="93.98" width="0.2032" layer="91"/>
-</segment>
-<segment>
 <wire x1="114.3" y1="149.86" x2="104.14" y2="149.86" width="0.2032" layer="91"/>
 <label x="104.14" y="149.86" size="1.778" layer="95"/>
@@
 <pinref part="U$1" gate="G$1" pin="A2"/>
 </segment>
+<segment>
+<label x="73.66" y="91.44" size="1.778" layer="95"/>
+<pinref part="BH" gate="ECOG$1" pin="SPI-CS@B3"/>
+<wire x1="73.66" y1="91.44" x2="99.06" y2="91.44" width="0.2032" layer="91"/>
+</segment>
 </net>
 <net name="D6/A4" class="0">
@@
 <net name="SPI-CS1" class="0">
 <segment>
-<label x="73.66" y="91.44" size="1.778" layer="95"/>
-<pinref part="BH" gate="ECOG$1" pin="SPI-CS@B3"/>
-<wire x1="73.66" y1="91.44" x2="99.06" y2="91.44" width="0.2032" layer="91"/>
-</segment>
-<segment>
 <wire x1="114.3" y1="137.16" x2="104.14" y2="137.16" width="0.2032" layer="91"/>
 <label x="104.14" y="137.16" size="1.778" layer="95"/>
 <pinref part="U$1" gate="G$1" pin="D4"/>
 </segment>
-</net>
+<segment>
+<label x="170.18" y="93.98" size="1.778" layer="95"/>
+<pinref part="AL" gate="ECOG$1" pin="SPI-CS@B3"/>
+<wire x1="182.88" y1="93.98" x2="157.48" y2="93.98" width="0.2032" layer="91"/>
+</segment>
+</net>

Commit message: V1.2
Moved JST battery connector
Parts:
- removed X100: JSTPH, microbuilder:CON_JST_PH_2PIN
Connections:
- net GND: no longer X100.1
- net VBAT: no longer X100.2
Changed lines of the file:
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@@
 <attribute name="PARTNO" value="MBR120VLSFT3G,on semiconductor,dk,MBR120VLSFT3GOSCT-ND ,DIODE SCHOTTKY 20V 1A SOD123FL , REF71"/>
-</part>
-<part name="X100" library="microbuilder" deviceset="CON_JST_PH_2PIN" device="" value="JSTPH">
-<attribute name="PARTNO" value="S2B-PH-SM4-TB(LF)(SN),JST SALES AMERICA INC (VA),dk,455-1749-1-ND,CONN HEADER PH SIDE 2POS 2MM SMD, REF69"/>
 </part>
 <part name="U$16" library="microbuilder" deviceset="VBAT" device=""/>
@@
 <attribute name="PARTNO" x="33.02" y="157.48" size="1.778" layer="96" display="off"/>
 </instance>
-<instance part="X100" gate="G$1" x="88.9" y="142.24" rot="R180">
-<attribute name="PARTNO" x="88.9" y="142.24" size="1.778" layer="96" display="off"/>
-</instance>
 <instance part="U$16" gate="G$1" x="91.44" y="152.4"/>
 <instance part="U$22" gate="G$1" x="91.44" y="129.54"/>
@@
 </segment>
 <segment>
-<pinref part="X100" gate="G$1" pin="1"/>
 <pinref part="U$22" gate="G$1" pin="GND"/>
 <wire x1="91.44" y1="132.08" x2="91.44" y2="139.7" width="0.1524" layer="91"/>
 <pinref part="JP1" gate="G$1" pin="1"/>
-<junction x="91.44" y="139.7"/>
 </segment>
 <segment>
@@
 </segment>
 <segment>
-<pinref part="X100" gate="G$1" pin="2"/>
 <pinref part="U$16" gate="G$1" pin="VBAT"/>
 <wire x1="91.44" y1="149.86" x2="91.44" y2="142.24" width="0.1524" layer="91"/>
 <pinref part="JP1" gate="G$1" pin="2"/>
-<junction x="91.44" y="142.24"/>
-</segment>
-<segment>
+</segment>
+<segment>

Commit message: V1.2.1
Fixed a problem with A0-A3
Parts:
- JP2, JP3: device SparkFun:M02POGO_PIN_HOLES_ONLY -> SparkFun:M021X02_NO_SILK
Connections:
- net D5/A5: now also U$1.A3; no longer U$1.A0
- net D6/A4: now also U$1.A2; no longer U$1.A1
- net D7/A3: now also U$1.A1; no longer U$1.A2
- net D8/A2: now also U$1.A0; no longer U$1.A3
Other:
- moved on the sheet: JP2, JP3
Changed lines of the file:
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@@
 <part name="3V3_PWR3" library="GadgetFactory" deviceset="3V3" device=""/>
 <part name="JP1" library="SparkFun" deviceset="M02" device="-JST-2-PTH-NO_SILK"/>
-<part name="JP2" library="SparkFun" deviceset="M02" device="POGO_PIN_HOLES_ONLY"/>
-<part name="JP3" library="SparkFun" deviceset="M02" device="POGO_PIN_HOLES_ONLY"/>
+<part name="JP2" library="SparkFun" deviceset="M02" device="1X02_NO_SILK"/>
+<part name="JP3" library="SparkFun" deviceset="M02" device="1X02_NO_SILK"/>
 </parts>
 <sheets>
@@
 <instance part="GND3" gate="A" x="129.54" y="170.18" rot="R180"/>
 <instance part="3V3_PWR3" gate="A" x="132.08" y="170.18"/>
-<instance part="JP2" gate="G$1" x="12.7" y="12.7"/>
-<instance part="JP3" gate="G$1" x="25.4" y="12.7"/>
+<instance part="JP2" gate="G$1" x="20.32" y="12.7"/>
+<instance part="JP3" gate="G$1" x="35.56" y="12.7"/>
 </instances>
 <busses>
@@
 </segment>
 <segment>
-<wire x1="152.4" y1="142.24" x2="162.56" y2="142.24" width="0.2032" layer="91"/>
-<label x="154.94" y="142.24" size="1.778" layer="95"/>
-<pinref part="U$1" gate="G$1" pin="A3"/>
-</segment>
-<segment>
 <wire x1="170.18" y1="50.8" x2="182.88" y2="50.8" width="0.2032" layer="91"/>
 <label x="170.18" y="50.8" size="1.778" layer="95"/>
 <pinref part="AH" gate="ECOG$1" pin="SPI-CS@B3"/>
 <wire x1="170.18" y1="50.8" x2="157.48" y2="50.8" width="0.1524" layer="91"/>
+</segment>
+<segment>
+<wire x1="152.4" y1="134.62" x2="162.56" y2="134.62" width="0.2032" layer="91"/>
+<label x="154.94" y="134.62" size="1.778" layer="95"/>
+<pinref part="U$1" gate="G$1" pin="A0"/>
 </segment>
 </net>
@@
 </segment>
 <segment>
-<wire x1="152.4" y1="139.7" x2="162.56" y2="139.7" width="0.2032" layer="91"/>
-<label x="154.94" y="139.7" size="1.778" layer="95"/>
-<pinref part="U$1" gate="G$1" pin="A2"/>
-</segment>
-<segment>
 <label x="73.66" y="91.44" size="1.778" layer="95"/>
 <pinref part="BH" gate="ECOG$1" pin="SPI-CS@B3"/>
 <wire x1="73.66" y1="91.44" x2="99.06" y2="91.44" width="0.2032" layer="91"/>
+</segment>
+<segment>
+<wire x1="152.4" y1="137.16" x2="162.56" y2="137.16" width="0.2032" layer="91"/>
+<label x="154.94" y="137.16" size="1.778" layer="95"/>
+<pinref part="U$1" gate="G$1" pin="A1"/>
 </segment>
 </net>
@@
 </segment>
 <segment>
-<wire x1="152.4" y1="137.16" x2="162.56" y2="137.16" width="0.2032" layer="91"/>
-<label x="154.94" y="137.16" size="1.778" layer="95"/>
-<pinref part="U$1" gate="G$1" pin="A1"/>
+<wire x1="152.4" y1="139.7" x2="162.56" y2="139.7" width="0.2032" layer="91"/>
+<label x="154.94" y="139.7" size="1.778" layer="95"/>
+<pinref part="U$1" gate="G$1" pin="A2"/>
 </segment>
 </net>
@@
 </segment>
 <segment>
-<wire x1="152.4" y1="134.62" x2="162.56" y2="134.62" width="0.2032" layer="91"/>
-<label x="154.94" y="134.62" size="1.778" layer="95"/>
-<pinref part="U$1" gate="G$1" pin="A0"/>
-</segment>
-</net>
+<wire x1="152.4" y1="142.24" x2="162.56" y2="142.24" width="0.2032" layer="91"/>
+<label x="154.94" y="142.24" size="1.778" layer="95"/>
+<pinref part="U$1" gate="G$1" pin="A3"/>
+</segment>
+</net>

Commit message: All the 2.0 updates
Connections:
- net D0/RX renamed D0/RX/MISO
- net D1/TX renamed D1/TX/MOSI
Changed lines of the file:
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@@
 </busses>
 <nets>
-<net name="D0/RX" class="0">
+<net name="D0/RX/MISO" class="0">
 <segment>
 <wire x1="119.38" y1="101.6" x2="139.7" y2="101.6" width="0.1524" layer="91"/>
@@
 <segment>
 <wire x1="114.3" y1="149.86" x2="104.14" y2="149.86" width="0.2032" layer="91"/>
-<label x="104.14" y="149.86" size="1.778" layer="95"/>
+<label x="103.632" y="150.114" size="1.778" layer="95"/>
 <pinref part="U$1" gate="G$1" pin="RX1"/>
 </segment>
@@
 </segment>
 </net>
-<net name="D1/TX" class="0">
+<net name="D1/TX/MOSI" class="0">
 <segment>
 <wire x1="121.92" y1="99.06" x2="139.7" y2="99.06" width="0.1524" layer="91"/>
@@
 <segment>
 <wire x1="114.3" y1="152.4" x2="104.14" y2="152.4" width="0.2032" layer="91"/>
-<label x="104.14" y="152.4" size="1.778" layer="95"/>
+<label x="103.632" y="152.4" size="1.778" layer="95"/>
 <pinref part="U$1" gate="G$1" pin="TX0"/>
 </segment>
