File: eCog100_ESP8266_Wifi.sch (EAGLE design)
At the start: 6 parts

Commit message: Latest updated to V1.4
Changed lines of the file:
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@@
 <instances>
 <instance part="FRAME1" gate="G$1" x="0" y="0"/>
-<instance part="GND2" gate="A" x="233.68" y="129.54" rot="R270"/>
-<instance part="ECOG" gate="ECOG_GENERAL" x="241.3" y="127"/>
+<instance part="GND2" gate="A" x="236.22" y="127"/>
+<instance part="ECOG" gate="ECOG_GENERAL" x="246.38" y="160.02" rot="MR180"/>
 <instance part="X1" gate="G$1" x="177.8" y="149.86"/>
 <instance part="R1" gate="A" x="200.66" y="167.64" rot="R90"/>
@@
 <net name="GND" class="0">
 <segment>
-<pinref part="ECOG" gate="ECOG_GENERAL" pin="GND"/>
-<pinref part="GND2" gate="A" pin="GND"/>
-</segment>
-<segment>
 <pinref part="R2" gate="A" pin="1"/>
 <pinref part="GND1" gate="A" pin="GND"/>
@@
 <wire x1="198.12" y1="137.16" x2="198.12" y2="121.92" width="0.2032" layer="91"/>
 </segment>
+<segment>
+<pinref part="ECOG" gate="ECOG_GENERAL" pin="GND"/>
+<wire x1="241.3" y1="157.48" x2="236.22" y2="157.48" width="0.1524" layer="91"/>
+<pinref part="GND2" gate="A" pin="GND"/>
+<wire x1="236.22" y1="157.48" x2="236.22" y2="129.54" width="0.1524" layer="91"/>
+</segment>
 </net>
 <net name="TX" class="0">
@@
 <label x="220.98" y="154.94" size="1.778" layer="95"/>
 <pinref part="X1" gate="G$1" pin="TXD"/>
-<wire x1="195.58" y1="154.94" x2="236.22" y2="154.94" width="0.2032" layer="91"/>
+<wire x1="195.58" y1="154.94" x2="241.3" y2="154.94" width="0.2032" layer="91"/>
 </segment>
 </net>
@@
 <label x="220.98" y="152.4" size="1.778" layer="95"/>
 <pinref part="X1" gate="G$1" pin="RXD"/>
-<wire x1="195.58" y1="152.4" x2="236.22" y2="152.4" width="0.2032" layer="91"/>
+<wire x1="195.58" y1="152.4" x2="241.3" y2="152.4" width="0.2032" layer="91"/>
 </segment>
 </net>
@@
 <wire x1="220.98" y1="101.6" x2="220.98" y2="147.32" width="0.2032" layer="91"/>
 <pinref part="ECOG" gate="ECOG_GENERAL" pin="G3"/>
-<wire x1="220.98" y1="147.32" x2="236.22" y2="147.32" width="0.2032" layer="91"/>
+<wire x1="220.98" y1="147.32" x2="241.3" y2="147.32" width="0.2032" layer="91"/>
 <pinref part="R3" gate="A" pin="1"/>
 <wire x1="147.32" y1="160.02" x2="147.32" y2="154.94" width="0.2032" layer="91"/>
@@
 <wire x1="205.74" y1="144.78" x2="205.74" y2="149.86" width="0.2032" layer="91"/>
 <pinref part="ECOG" gate="ECOG_GENERAL" pin="G2"/>
-<wire x1="205.74" y1="149.86" x2="236.22" y2="149.86" width="0.2032" layer="91"/>
+<wire x1="205.74" y1="149.86" x2="241.3" y2="149.86" width="0.2032" layer="91"/>
 <label x="205.74" y="149.86" size="1.778" layer="95"/>
 </segment>
@@
 <pinref part="ECOG" gate="ECOG_GENERAL" pin="3V3"/>
 <pinref part="3V3_PWR5" gate="A" pin="3V3"/>
-<wire x1="236.22" y1="134.62" x2="231.14" y2="134.62" width="0.2032" layer="91"/>
+<wire x1="241.3" y1="134.62" x2="231.14" y2="134.62" width="0.2032" layer="91"/>
 <wire x1="231.14" y1="134.62" x2="231.14" y2="162.56" width="0.2032" layer="91"/>
 </segment>

Commit message: Added parts to attributes for BOM
Parts:
- R1, R2, R3, R4: DIGIKEY (none) -> RMCF0805JT10K0CT-ND
- X1: ADAFRUIT (none) -> 2491
Changed lines of the file:
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@@
 <part name="GND2" library="GadgetFactory" deviceset="GND" device=""/>
 <part name="ECOG" library="eCogs" deviceset="ECOG_GENERAL_ROW" device="ECOG_GENERAL_SMD" value="ECOG_GENERAL_ROWECOG_GENERAL_SMD"/>
-<part name="X1" library="adafruit" deviceset="ESP-12" device=""/>
-<part name="R1" library="GadgetFactory" deviceset="R" device="0805" value="10K"/>
-<part name="R2" library="GadgetFactory" deviceset="R" device="0805" value="10K"/>
-<part name="R3" library="GadgetFactory" deviceset="R" device="0805" value="10K"/>
-<part name="R4" library="GadgetFactory" deviceset="R" device="0805" value="10K"/>
+<part name="X1" library="adafruit" deviceset="ESP-12" device="">
+<attribute name="ADAFRUIT" value="2491"/>
+</part>
+<part name="R1" library="GadgetFactory" deviceset="R" device="0805" value="10K">
+<attribute name="DIGIKEY" value="RMCF0805JT10K0CT-ND"/>
+</part>
+<part name="R2" library="GadgetFactory" deviceset="R" device="0805" value="10K">
+<attribute name="DIGIKEY" value="RMCF0805JT10K0CT-ND"/>
+</part>
+<part name="R3" library="GadgetFactory" deviceset="R" device="0805" value="10K">
+<attribute name="DIGIKEY" value="RMCF0805JT10K0CT-ND"/>
+</part>
+<part name="R4" library="GadgetFactory" deviceset="R" device="0805" value="10K">
+<attribute name="DIGIKEY" value="RMCF0805JT10K0CT-ND"/>
+</part>
 <part name="GND1" library="GadgetFactory" deviceset="GND" device=""/>
 <part name="3V3_PWR1" library="GadgetFactory" deviceset="3V3" device=""/>
@@
 <instance part="GND2" gate="A" x="236.22" y="127"/>
 <instance part="ECOG" gate="ECOG_GENERAL" x="246.38" y="160.02" rot="MR180"/>
-<instance part="X1" gate="G$1" x="177.8" y="149.86"/>
-<instance part="R1" gate="A" x="200.66" y="167.64" rot="R90"/>
-<instance part="R2" gate="A" x="208.28" y="127" rot="R90"/>
-<instance part="R3" gate="A" x="147.32" y="165.1" rot="R90"/>
-<instance part="R4" gate="A" x="152.4" y="165.1" rot="R90"/>
+<instance part="X1" gate="G$1" x="177.8" y="149.86">
+<attribute name="ADAFRUIT" x="177.8" y="149.86" size="1.778" layer="96" display="off"/>
+</instance>
+<instance part="R1" gate="A" x="200.66" y="167.64" rot="R90">
+<attribute name="DIGIKEY" x="200.66" y="167.64" size="1.778" layer="96" rot="R90" display="off"/>
+</instance>
+<instance part="R2" gate="A" x="208.28" y="127" rot="R90">
+<attribute name="DIGIKEY" x="208.28" y="127" size="1.778" layer="96" rot="R90" display="off"/>
+</instance>
+<instance part="R3" gate="A" x="147.32" y="165.1" rot="R90">
+<attribute name="DIGIKEY" x="147.32" y="165.1" size="1.778" layer="96" rot="R90" display="off"/>
+</instance>
+<instance part="R4" gate="A" x="152.4" y="165.1" rot="R90">
+<attribute name="DIGIKEY" x="152.4" y="165.1" size="1.778" layer="96" rot="R90" display="off"/>
+</instance>
 <instance part="GND1" gate="A" x="208.28" y="119.38"/>
 <instance part="3V3_PWR1" gate="A" x="147.32" y="172.72"/>

Commit message: All the 2.0 updates
Connections:
- net RX renamed RX/MOSI
- net TX renamed TX/MISO
Changed lines of the file:
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@@
 </segment>
 </net>
-<net name="TX" class="0">
+<net name="TX/MISO" class="0">
 <segment>
 <pinref part="ECOG" gate="ECOG_GENERAL" pin="G0"/>
-<label x="220.98" y="154.94" size="1.778" layer="95"/>
+<label x="218.44" y="154.94" size="1.778" layer="95"/>
 <pinref part="X1" gate="G$1" pin="TXD"/>
 <wire x1="195.58" y1="154.94" x2="241.3" y2="154.94" width="0.2032" layer="91"/>
 </segment>
 </net>
-<net name="RX" class="0">
+<net name="RX/MOSI" class="0">
 <segment>
 <pinref part="ECOG" gate="ECOG_GENERAL" pin="G1"/>
-<label x="220.98" y="152.4" size="1.778" layer="95"/>
+<label x="218.44" y="152.4" size="1.778" layer="95"/>
 <pinref part="X1" gate="G$1" pin="RXD"/>
 <wire x1="195.58" y1="152.4" x2="241.3" y2="152.4" width="0.2032" layer="91"/>
