File: eCog103_Sensor.sch (EAGLE design)
At the start: 1 part

Commit message: V1.1
Parts:
- added U$1: SENSOR, eCogs:SENSOR
Connections:
- new net A1: ECOG.G0, U$1.DO/S
- new net A2: ECOG.G1, U$1.AO
- new net A3: ECOG.G2
- net 3V3: now also U$1.+
- net GND: now also U$1.GND
Other:
- note added: "An Analog eCog will only work on AH and BH."
- moved on the sheet: ECOG
Changed lines of the file:
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@@
 <layer number="54" name="bGND_GNDA" color="1" fill="9" visible="no" active="no"/>
 <layer number="56" name="wert" color="3" fill="1" visible="no" active="no"/>
+<layer number="57" name="tCAD" color="7" fill="1" visible="no" active="no"/>
+<layer number="59" name="tCarbon" color="7" fill="1" visible="no" active="no"/>
+<layer number="60" name="bCarbon" color="7" fill="1" visible="no" active="no"/>
+<layer number="90" name="Modules" color="7" fill="1" visible="yes" active="yes"/>
 <layer number="91" name="Nets" color="2" fill="1" visible="yes" active="yes"/>
 <layer number="92" name="Busses" color="1" fill="1" visible="yes" active="yes"/>
@@
 <layer number="97" name="Info" color="7" fill="1" visible="yes" active="yes"/>
 <layer number="98" name="Guide" color="6" fill="1" visible="yes" active="yes"/>
+<layer number="99" name="SpiceOrder" color="7" fill="1" visible="no" active="no"/>
 <layer number="100" name="Muster" color="7" fill="1" visible="no" active="no"/>
 <layer number="101" name="Patch_Top" color="12" fill="4" visible="no" active="yes"/>
@@
 <layer number="111" name="tGTest" color="7" fill="1" visible="yes" active="yes"/>
 <layer number="112" name="bGTest" color="7" fill="1" visible="yes" active="yes"/>
+<layer number="113" name="ReferenceLS" color="7" fill="1" visible="no" active="no"/>
 <layer number="116" name="Patch_BOT" color="9" fill="4" visible="no" active="yes"/>
+<layer number="118" name="Rect_Pads" color="7" fill="1" visible="no" active="no"/>
 <layer number="121" name="_tsilk" color="7" fill="1" visible="yes" active="yes"/>
 <layer number="122" name="_bsilk" color="7" fill="1" visible="no" active="yes"/>
@@
 <layer number="124" name="bTestmark" color="7" fill="1" visible="yes" active="yes"/>
 <layer number="125" name="_tNames" color="7" fill="1" visible="yes" active="yes"/>
+<layer number="126" name="_bNames" color="7" fill="1" visible="yes" active="yes"/>
+<layer number="127" name="_tValues" color="7" fill="1" visible="yes" active="yes"/>
+<layer number="128" name="_bValues" color="7" fill="1" visible="yes" active="yes"/>
+<layer number="129" name="Mask" color="7" fill="1" visible="yes" active="yes"/>
 <layer number="131" name="prix" color="7" fill="1" visible="no" active="yes"/>
 <layer number="132" name="test" color="7" fill="1" visible="no" active="yes"/>
@@
 <layer number="135" name="Port3" color="7" fill="1" visible="yes" active="yes"/>
 <layer number="144" name="Drill_legend" color="7" fill="1" visible="yes" active="yes"/>
+<layer number="150" name="Notes" color="7" fill="1" visible="yes" active="yes"/>
 <layer number="151" name="HeatSink" color="7" fill="1" visible="no" active="yes"/>
+<layer number="152" name="_bDocu" color="7" fill="1" visible="yes" active="yes"/>
+<layer number="153" name="FabDoc1" color="6" fill="1" visible="no" active="no"/>
+<layer number="154" name="FabDoc2" color="2" fill="1" visible="no" active="no"/>
+<layer number="155" name="FabDoc3" color="7" fill="15" visible="no" active="no"/>
 <layer number="199" name="Contour" color="7" fill="1" visible="yes" active="yes"/>
 <layer number="200" name="200bmp" color="1" fill="10" visible="no" active="no"/>
@@
 <layer number="223" name="223bmp" color="24" fill="1" visible="no" active="no"/>
 <layer number="224" name="224bmp" color="25" fill="1" visible="no" active="no"/>
+<layer number="225" name="225bmp" color="7" fill="1" visible="yes" active="yes"/>
+<layer number="226" name="226bmp" color="7" fill="1" visible="yes" active="yes"/>
+<layer number="227" name="227bmp" color="7" fill="1" visible="yes" active="yes"/>
+<layer number="228" name="228bmp" color="7" fill="1" visible="yes" active="yes"/>
+<layer number="229" name="229bmp" color="7" fill="1" visible="yes" active="yes"/>
+<layer number="230" name="230bmp" color="7" fill="1" visible="yes" active="yes"/>
+<layer number="231" name="Eagle3D_PG1" color="7" fill="1" visible="no" active="no"/>
+<layer number="232" name="Eagle3D_PG2" color="7" fill="1" visible="no" active="no"/>
+<layer number="233" name="Eagle3D_PG3" color="7" fill="1" visible="no" active="no"/>
+<layer number="248" name="Housing" color="7" fill="1" visible="yes" active="yes"/>
+<layer number="249" name="Edge" color="7" fill="1" visible="yes" active="yes"/>
 <layer number="250" name="Descript" color="3" fill="1" visible="no" active="no"/>
 <layer number="251" name="SMDround" color="4" fill="9" visible="no" active="yes"/>
 <layer number="254" name="cooling" color="7" fill="1" visible="no" active="yes"/>
+<layer number="255" name="routoute" color="7" fill="1" visible="yes" active="yes"/>
 </layers>
 <schematic xreflabel="%F%N/%S.%C%R" xrefpart="/%S.%C%R">
@@
 <part name="3V3_PWR1" library="eCogs" deviceset="3V3" device=""/>
 <part name="GND1" library="eCogs" deviceset="GND" device=""/>
+<part name="U$1" library="eCogs" deviceset="SENSOR" device=""/>
+<part name="3V3_PWR2" library="eCogs" deviceset="3V3" device=""/>
+<part name="GND2" library="eCogs" deviceset="GND" device=""/>
 </parts>
 <sheets>
@@
 <text x="317.5" y="30.48" size="2.1844" layer="91">Copyright 2016 Gadget Factory, LLC</text>
 <text x="317.5" y="25.4" size="1.778" layer="91">See more details at www.GadgetFactory.net</text>
+<text x="68.58" y="22.86" size="6.4516" layer="91">An Analog eCog will only work on AH and BH.</text>
 </plain>
 <instances>
 <instance part="FRAME1" gate="G$1" x="0" y="0"/>
-<instance part="ECOG" gate="ECOG_GENERAL" x="55.88" y="53.34"/>
-<instance part="3V3_PWR1" gate="A" x="35.56" y="63.5"/>
-<instance part="GND1" gate="A" x="35.56" y="50.8"/>
+<instance part="ECOG" gate="ECOG_GENERAL" x="350.52" y="60.96"/>
+<instance part="3V3_PWR1" gate="A" x="330.2" y="71.12"/>
+<instance part="GND1" gate="A" x="330.2" y="58.42"/>
+<instance part="U$1" gate="SENSOR" x="287.02" y="76.2"/>
+<instance part="3V3_PWR2" gate="A" x="281.94" y="91.44"/>
+<instance part="GND2" gate="A" x="281.94" y="71.12"/>
 </instances>
 <busses>
@@
 <pinref part="ECOG" gate="ECOG_GENERAL" pin="3V3"/>
 <pinref part="3V3_PWR1" gate="A" pin="3V3"/>
-<wire x1="50.8" y1="60.96" x2="35.56" y2="60.96" width="0.2032" layer="91"/>
+<wire x1="345.44" y1="68.58" x2="330.2" y2="68.58" width="0.2032" layer="91"/>
+</segment>
+<segment>
+<pinref part="U$1" gate="SENSOR" pin="+"/>
+<pinref part="3V3_PWR2" gate="A" pin="3V3"/>
+<wire x1="292.1" y1="83.82" x2="281.94" y2="83.82" width="0.2032" layer="91"/>
+<wire x1="281.94" y1="83.82" x2="281.94" y2="88.9" width="0.2032" layer="91"/>
 </segment>
 </net>
@@
 <pinref part="ECOG" gate="ECOG_GENERAL" pin="GND"/>
 <pinref part="GND1" gate="A" pin="GND"/>
-<wire x1="50.8" y1="55.88" x2="35.56" y2="55.88" width="0.2032" layer="91"/>
-<wire x1="35.56" y1="55.88" x2="35.56" y2="53.34" width="0.2032" layer="91"/>
+<wire x1="345.44" y1="63.5" x2="330.2" y2="63.5" width="0.2032" layer="91"/>
+<wire x1="330.2" y1="63.5" x2="330.2" y2="60.96" width="0.2032" layer="91"/>
+</segment>
+<segment>
+<pinref part="U$1" gate="SENSOR" pin="GND"/>
+<pinref part="GND2" gate="A" pin="GND"/>
+<wire x1="292.1" y1="81.28" x2="281.94" y2="81.28" width="0.2032" layer="91"/>
+<wire x1="281.94" y1="81.28" x2="281.94" y2="73.66" width="0.2032" layer="91"/>
+</segment>
+</net>
+<net name="A1" class="0">
+<segment>
+<pinref part="ECOG" gate="ECOG_GENERAL" pin="G0"/>
+<label x="335.28" y="88.9" size="1.778" layer="95"/>
+<pinref part="U$1" gate="SENSOR" pin="DO/S"/>
+<wire x1="292.1" y1="86.36" x2="309.88" y2="86.36" width="0.2032" layer="91"/>
+<wire x1="309.88" y1="86.36" x2="309.88" y2="88.9" width="0.2032" layer="91"/>
+<wire x1="309.88" y1="88.9" x2="345.44" y2="88.9" width="0.2032" layer="91"/>
+</segment>
+</net>
+<net name="A2" class="0">
+<segment>
+<pinref part="ECOG" gate="ECOG_GENERAL" pin="G1"/>
+<label x="335.28" y="86.36" size="1.778" layer="95"/>
+<pinref part="U$1" gate="SENSOR" pin="AO"/>
+<wire x1="292.1" y1="78.74" x2="312.42" y2="78.74" width="0.2032" layer="91"/>
+<wire x1="312.42" y1="78.74" x2="312.42" y2="86.36" width="0.2032" layer="91"/>
+<wire x1="312.42" y1="86.36" x2="345.44" y2="86.36" width="0.2032" layer="91"/>
+</segment>
+</net>
+<net name="A3" class="0">
+<segment>
+<pinref part="ECOG" gate="ECOG_GENERAL" pin="G2"/>
+<wire x1="345.44" y1="83.82" x2="335.28" y2="83.82" width="0.2032" layer="91"/>
+<label x="335.28" y="83.82" size="1.778" layer="95"/>
 </segment>
 </net>
@@
 </schematic>
 </drawing>
+<compatibility>
+<note version="6.3" minversion="6.2.2" severity="warning">
+Since Version 6.2.2 text objects can contain more than one line,
+which will not be processed correctly with this version.
+</note>
+</compatibility>
 </eagle>

Commit message: Latest updated to V1.4
Connections:
- removed net A3: ECOG.G2
- net A1: now also U$1.AO; no longer U$1.DO/S
- net A2: now also U$1.DO/S; no longer U$1.AO
Changed lines of the file:
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@@
 <text x="317.5" y="30.48" size="2.1844" layer="91">Copyright 2016 Gadget Factory, LLC</text>
 <text x="317.5" y="25.4" size="1.778" layer="91">See more details at www.GadgetFactory.net</text>
-<text x="68.58" y="22.86" size="6.4516" layer="91">An Analog eCog will only work on AH and BH.</text>
+<text x="27.94" y="22.86" size="6.4516" layer="91">An Analog eCog will only work on AH and BH.</text>
 </plain>
 <instances>
 <instance part="FRAME1" gate="G$1" x="0" y="0"/>
 <instance part="ECOG" gate="ECOG_GENERAL" x="350.52" y="60.96"/>
-<instance part="3V3_PWR1" gate="A" x="330.2" y="71.12"/>
-<instance part="GND1" gate="A" x="330.2" y="58.42"/>
+<instance part="3V3_PWR1" gate="A" x="345.44" y="93.98"/>
+<instance part="GND1" gate="A" x="345.44" y="50.8"/>
 <instance part="U$1" gate="SENSOR" x="287.02" y="76.2"/>
 <instance part="3V3_PWR2" gate="A" x="281.94" y="91.44"/>
@@
 <net name="3V3" class="0">
 <segment>
-<pinref part="ECOG" gate="ECOG_GENERAL" pin="3V3"/>
-<pinref part="3V3_PWR1" gate="A" pin="3V3"/>
-<wire x1="345.44" y1="68.58" x2="330.2" y2="68.58" width="0.2032" layer="91"/>
-</segment>
-<segment>
 <pinref part="U$1" gate="SENSOR" pin="+"/>
 <pinref part="3V3_PWR2" gate="A" pin="3V3"/>
 <wire x1="292.1" y1="83.82" x2="281.94" y2="83.82" width="0.2032" layer="91"/>
 <wire x1="281.94" y1="83.82" x2="281.94" y2="88.9" width="0.2032" layer="91"/>
+</segment>
+<segment>
+<pinref part="ECOG" gate="ECOG_GENERAL" pin="3V3"/>
+<pinref part="3V3_PWR1" gate="A" pin="3V3"/>
+<wire x1="345.44" y1="91.44" x2="345.44" y2="86.36" width="0.1524" layer="91"/>
 </segment>
 </net>
@@
 <pinref part="ECOG" gate="ECOG_GENERAL" pin="GND"/>
 <pinref part="GND1" gate="A" pin="GND"/>
-<wire x1="345.44" y1="63.5" x2="330.2" y2="63.5" width="0.2032" layer="91"/>
-<wire x1="330.2" y1="63.5" x2="330.2" y2="60.96" width="0.2032" layer="91"/>
+<wire x1="345.44" y1="63.5" x2="345.44" y2="53.34" width="0.2032" layer="91"/>
 </segment>
 <segment>
@@
 </segment>
 </net>
+<net name="A2" class="0">
+<segment>
+<pinref part="U$1" gate="SENSOR" pin="DO/S"/>
+<wire x1="292.1" y1="86.36" x2="314.96" y2="86.36" width="0.2032" layer="91"/>
+<pinref part="ECOG" gate="ECOG_GENERAL" pin="G1"/>
+<wire x1="345.44" y1="68.58" x2="314.96" y2="68.58" width="0.2032" layer="91"/>
+<wire x1="314.96" y1="68.58" x2="314.96" y2="86.36" width="0.2032" layer="91"/>
+<label x="330.2" y="68.58" size="1.778" layer="95"/>
+</segment>
+</net>
 <net name="A1" class="0">
 <segment>
+<pinref part="U$1" gate="SENSOR" pin="AO"/>
+<wire x1="292.1" y1="78.74" x2="312.42" y2="78.74" width="0.2032" layer="91"/>
 <pinref part="ECOG" gate="ECOG_GENERAL" pin="G0"/>
-<label x="335.28" y="88.9" size="1.778" layer="95"/>
-<pinref part="U$1" gate="SENSOR" pin="DO/S"/>
-<wire x1="292.1" y1="86.36" x2="309.88" y2="86.36" width="0.2032" layer="91"/>
-<wire x1="309.88" y1="86.36" x2="309.88" y2="88.9" width="0.2032" layer="91"/>
-<wire x1="309.88" y1="88.9" x2="345.44" y2="88.9" width="0.2032" layer="91"/>
+<wire x1="345.44" y1="66.04" x2="312.42" y2="66.04" width="0.2032" layer="91"/>
+<wire x1="312.42" y1="66.04" x2="312.42" y2="78.74" width="0.2032" layer="91"/>
+<label x="330.2" y="66.04" size="1.778" layer="95"/>
 </segment>
 </net>
-<net name="A2" class="0">
-<segment>
-<pinref part="ECOG" gate="ECOG_GENERAL" pin="G1"/>
-<label x="335.28" y="86.36" size="1.778" layer="95"/>
-<pinref part="U$1" gate="SENSOR" pin="AO"/>
-<wire x1="292.1" y1="78.74" x2="312.42" y2="78.74" width="0.2032" layer="91"/>
-<wire x1="312.42" y1="78.74" x2="312.42" y2="86.36" width="0.2032" layer="91"/>
-<wire x1="312.42" y1="86.36" x2="345.44" y2="86.36" width="0.2032" layer="91"/>
-</segment>
-</net>
-<net name="A3" class="0">
-<segment>
-<pinref part="ECOG" gate="ECOG_GENERAL" pin="G2"/>
-<wire x1="345.44" y1="83.82" x2="335.28" y2="83.82" width="0.2032" layer="91"/>
-<label x="335.28" y="83.82" size="1.778" layer="95"/>
-</segment>
-</net>

Commit message: All the 2.0 updates
Other:
- note added: "An Analog eCog will only work on A and D."
- note removed: "An Analog eCog will only work on AH and BH."
Changed lines of the file:
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@@
 <text x="317.5" y="30.48" size="2.1844" layer="91">Copyright 2016 Gadget Factory, LLC</text>
 <text x="317.5" y="25.4" size="1.778" layer="91">See more details at www.GadgetFactory.net</text>
-<text x="27.94" y="22.86" size="6.4516" layer="91">An Analog eCog will only work on AH and BH.</text>
+<text x="27.94" y="22.86" size="6.4516" layer="91">An Analog eCog will only work on A and D.</text>
 </plain>
 <instances>
