File: eCog104_Joystick_PSP_Slide.sch (EAGLE design)
At the start: 2 parts

Commit message: All the 2.0 updates
Other:
- note added: "An Analog eCog will only work on A and D."
- note removed: "An Analog eCog will only work on AH and BH."
Changed lines of the file:
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@@
 <text x="317.5" y="30.48" size="2.1844" layer="91">Copyright 2016 Gadget Factory, LLC</text>
 <text x="317.5" y="25.4" size="1.778" layer="91">See more details at www.GadgetFactory.net</text>
-<text x="33.02" y="22.86" size="6.4516" layer="91">An Analog eCog will only work on AH and BH.</text>
+<text x="33.02" y="22.86" size="6.4516" layer="91">An Analog eCog will only work on A and D.</text>
 </plain>
 <instances>
