File: eCog106_BLED.sch (EAGLE design)
At the start: 17 parts, among them SW1 SPST_TACT-EVQQ2, SW2 SPST_TACT-EVQQ2, SW3 SPST_TACT-EVQQ2, SW4 SPST_TACT-EVQQ2

Commit message: Latest updated to V1.4
Parts:
- removed SW1, SW2, SW3, SW4: SPST_TACT-EVQQ2, adafruit:SPST_TACT-EVQQ2
- added S1, S2, S3, S4: (no value), SparkFun:TAC_SWITCHPTH
Connections:
- net 1: now also S1.1, S1.2
- net 2: now also S2.1, S2.2
- net 3: now also S3.1, S3.2
- net 3V3: now also S1.3, S1.4, S2.3, S2.4, S3.3, S3.4, S4.3, S4.4; no longer SW1.S1, SW2.S1, SW3.S1, SW4.S1
- net 4: now also S4.1, S4.2
Other:
- moved on the sheet: LED1, LED2, LED3, LED4, R1, R2, R3, R4, R5, R6, R7, R8

Commit message: Added parts to attributes for BOM
Parts:
- LED1, LED2, LED3, LED4: DIGIKEY (none) -> 475-1410-2-ND
- R1, R3, R5, R7: DIGIKEY (none) -> RMCF0805JT390RCT-ND
- R2, R4, R6, R8: DIGIKEY (none) -> RMCF0805JT10K0CT-ND
- S1, S2, S3, S4: DIGIKEY (none) -> 679-2428-ND
