File: eCog111_16ch_PWM_Servo.brd (EAGLE design)
At the start: 47.5 x 28 mm, 4 parts

Commit message: All the 2.0 updates
Parts:
- moved JP2 1.27 mm to (2.54, 14.0)
Routing:
- net N$3: track 49.1 -> 44.2 mm
- net N$2: track 47.8 -> 44.0 mm
- net N$1: track 45.6 -> 47.6 mm, vias 0 -> 2
- net 3V3: track 2.18 -> 4.09 mm
Other:
- outline, holes or cut-outs redrawn
- board text added: "ecog111 v2.0"
- board text removed: "ecog111 v1.0"
