File: eCog113_BLE_Bluetooth_HM10.brd (EAGLE design)
At the start: 47.5 x 28 mm, 3 parts

Commit message: All the 2.0 updates
Parts:
- added E1: HM-10-BOARD, JNHuaMao:26.9X13X2.2_BOARD
- added U$3: (no value), eCogs:LEGEND_DIO
- U$1: device ohw-logo:OSHW_FILLX350_NOTEXT -> GadgetFactory:GADGETBOX_TEXT
- U$2: device GadgetFactory:GADGETBOX_TEXT -> eCogs:LEGEND_DIO
- moved U$2 24.6 mm to (47.0, 7.62)
- moved U$1 17.6 mm to (24.1, 17.8)
Connections:
- new net RX/MOSI: E1.2, ECOG.G1
- new net TX/MISO: E1.1, ECOG.G0
- net 3V3: now also E1.11, E1.12
- net GND: now also E1.13, E1.14, E1.21, E1.22
Routing:
- net TX/MISO: track 0.00 -> 31.9 mm
- net RX/MOSI: track 0.00 -> 25.8 mm
- net 3V3: track 0.00 -> 7.62 mm, vias 0 -> 2
- net GND: track 2.88 -> 0.00 mm, vias 1 -> 0
- added copper zone on layer 1, net 3V3
- added copper zone on layer 16, net GND
- removed copper zone on layer 1, net GND
Other:
- board text added: "3.3V"
- board text added: "BLE Bluetooth (HM-10)"
- board text added: "GND"
- board text added: "RX/MOSI"
- board text added: "TX/MISO"
- board text added: "ecog113 v2.0"
- board text added: "ecog113.GadgetFactory.net"
- board text removed: "Blank"
- board text removed: "ecog0 v2.0"
- board text removed: "ecog0.GadgetFactory.net"
