File: pCog102_Wifi_PSPJoy_BLED_TFT.sch (EAGLE design)
At the start: 27 parts

Commit message: All the 2.0 updates
Parts:
- ECOG2: value ECOG_GENERAL_ROWECOG_GENERAL_SMD -> ECOG_BUSES_ROWECOG_BUSES_SMD; device eCogs:ECOG_GENERAL_ROWECOG_GENERAL_SMD -> eCogs:ECOG_BUSES_ROWECOG_BUSES_SMD
- ECOG3: value ECOG_BUSES_ROWECOG_BUSES_SMD -> ECOG_GENERAL_ROWECOG_GENERAL_SMD; device eCogs:ECOG_BUSES_ROWECOG_BUSES_SMD -> eCogs:ECOG_GENERAL_ROWECOG_GENERAL_SMD
- R1, R3: value 10K -> 390; DIGIKEY RMCF0805JT10K0CT-ND -> RMCF0805JT390RCT-ND
- R10, R12, R2, R4: DIGIKEY RMCF0805JT10K0CT-ND -> RMCF0805JT10K0CT-ND
- R11, R9: value 390 -> 10K; DIGIKEY RMCF0805JT390RCT-ND -> RMCF0805JT10K0CT-ND
- renumbered U$6 to U$7
Connections:
- removed net N$5: R4A.1, X1.CH_PD
- removed net N$6: LED1.A, R5A.2
- removed net RX: ECOG.G1, X1.RXD
- removed net TX: ECOG.G0, X1.TXD
- new net N$1: LED1.A, R1A.2
- new net N$2: LED2.A, R3A.2
- new net RX/MOSI: ECOG3.G1, X1.RXD
- new net TX/MISO: ECOG3.G0, X1.TXD
- net 1: now also ECOG.G0, R1A.1, R2A.2; no longer ECOG2.G0, R5A.1, R6A.2
- net 2: now also ECOG.G1, R3A.1, R4A.2; no longer ECOG2.G1, R7A.1, R8A.2
- net 3: now also ECOG.G2, R5A.1, R6A.2; no longer ECOG2.G2, R10A.2, R9A.1
- net 3V3: now also ECOG2.3V3@B8, ECOG3.3V3, R11A.2, R12A.2, R9A.2; no longer ECOG2.3V3, ECOG3.3V3@B8, R1A.2, R3A.2, R4A.2
- net 4: now also ECOG.G3, R7A.1, R8A.2; no longer ECOG2.G3, R11A.1, R12A.2
- net GND: now also ECOG2.GND@B, ECOG3.GND, R4A.1; no longer ECOG2.GND, ECOG3.GND@B, R12A.1
- net GPIO0/BOOTLOAD: now also ECOG3.G2; no longer ECOG.G2
- net N$10: now also R10A.2, X1.GPIO15; no longer ECOG3.I2C-SDA@B4, JP1.4
- net N$11: now also R12A.1, X1.CH_PD; no longer ECOG3.I2C-SCL@B5, JP1.3
- net N$3: now also LED3.A, R5A.2; no longer R1A.1, X1.GPIO2
- net N$4: now also LED4.A, R7A.2; no longer R2A.2, X1.GPIO15
- net N$7: now also ECOG2.I2C-SDA@B4, JP1.4; no longer LED2.A, R7A.2
- net N$8: now also ECOG2.I2C-SCL@B5, JP1.3; no longer LED3.A, R9A.2
- net N$9: now also R9A.1, X1.GPIO2; no longer LED4.A, R11A.2
- net RESET: now also ECOG3.G3, R11A.1; no longer ECOG.G3, R3A.1
Other:
- note added: "An Analog eCog will only work on A and D."
- note removed: "An Analog eCog will only work on AH and BH."
