File: GadgetBox-atmega32u4/Gadget-Box.brd (EAGLE design)
At the start: 93.5 x 53.5 mm, 44 parts, among them U1 MCP73831T-2ACI/OT, U2 AP2112-3.3, U3 ATMEGA32U4-XUAU, U4 ATMEGA32U4-XUMU, X1 CRYSTAL-0500290P1, X100 JSTPH

Commit message: Reorganized
Connections:
- net D0/RX renamed D0/RX/MISO
- net D1/TX renamed D1/TX/MISO
Changed lines of the file:
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@@
 <layer number="155" name="FabDoc3" color="7" fill="15" visible="no" active="no"/>
 <layer number="199" name="Contour" color="7" fill="1" visible="no" active="yes"/>
-<layer number="200" name="200bmp" color="1" fill="1" visible="yes" active="yes"/>
+<layer number="200" name="200bmp" color="1" fill="1" visible="no" active="yes"/>
 <layer number="201" name="201bmp" color="7" fill="1" visible="no" active="yes"/>
 <layer number="202" name="202bmp" color="7" fill="1" visible="no" active="yes"/>
@@
 <wire x1="68.618" y1="31.712" x2="68.58" y2="31.75" width="0.254" layer="1"/>
 </signal>
-<signal name="D1/TX">
+<signal name="D1/TX/MISO">
 <contactref element="U4" pad="21"/>
 <contactref element="U3" pad="21"/>
@@
 <wire x1="39.37" y1="8.89" x2="39.37" y2="10.16" width="0.254" layer="1"/>
 </signal>
-<signal name="D0/RX">
+<signal name="D0/RX/MISO">
 <contactref element="U4" pad="20"/>
 <contactref element="U3" pad="20"/>
