File: GadgetBox-mini-pro/Gadget-Box-mini-pro.brd (EAGLE design)
At the start: 93.5 x 53.5 mm, 27 parts, among them U1 MCP73831T-2ACI/OT, U2 AP2112-3.3

Commit message: Reorganized
Parts:
- R4, R7: device GadgetFactory:0805 -> GadgetFactory:0603
