File: eCogs/pCog100_Wifi_Sensor_uSD_TFT.brd (EAGLE design)
At the start: 47.5 x 28 mm, 30 parts

Commit message: Reorganized
Other:
- board text added: "XC0"
- board text added: "XC1"
- board text added: "XC2"
- board text added: "XC3"
- board text removed: "0"
- board text removed: "1"
- board text removed: "2"
- board text removed: "3"
