File: eCogs/pCog100_Wifi_Sensor_uSD_TFT.sch (EAGLE design)
At the start: 15 parts

Commit message: Reorganized
Parts:
- ECOG, ECOG1, ECOG2, ECOG3: PARTNO (none) -> NREC010SABC-M30RC,SULLINS CONNECTOR SOLUTIONS,dk,S1013EC-10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
- JP1: PARTNO (none) -> 346540,unknown,seeed,346540,"0.96"" 128*64 I2C Interface Wh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
- R1, R2, R3: PARTNO RMCF0805JT47K0 -> RMCF0805JT47K0,Stackpole Electronics Inc,DK,RMCF0805JT47K0C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
- R4, R5, R6, R7: PARTNO (none) -> RC0805JR-0710KL,YAGEO (VA),dk,311-10KARCT-ND,RES SMD 10K OH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
- SD1: PARTNO 101-00660-68-6 -> 101-00660-68-6,Amphenol,dk,101-00660-68-6-1-ND,Secure Digit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
- U$5: BOM (none) -> EXCLUDE
- X1: PARTNO (none) -> 385646,AI-Thinker,dx.com,385646,ESP8266 Serial Wi-Fi Wirele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
