File: eCogs/pCog101_Wifi_Remote_BLED.sch (EAGLE design)
At the start: 32 parts, among them T1 MMBT3904LT1G, T3 MMBT3904LT1G, U1 PNA460XM

Commit message: Reorganized
Parts:
- ECOG, ECOG1, ECOG2, ECOG3: PARTNO (none) -> NREC010SABC-M30RC,SULLINS CONNECTOR SOLUTIONS,dk,S1013EC-10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
- IR1, IR2: PARTNO (none) -> IR333C/H0/L10,everlight,dk,1080-1082-ND,EMITTER IR 940NM 10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
- JP1: PARTNO (none) -> 346540,unknown,dx.com,346540,"0.96"" 128*64 I2C Interface W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
- LED1, LED2, LED3, LED4: PARTNO (none) -> LTST-C170KGKT,LITE-ON INC (VA),DK,160-1414-1-ND,LED GREEN C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
- R1: PARTNO (none) -> RC0805JR-071KL,YAGEO (VA),dk,311-1.0KARCT-ND,RES SMD 1K OHM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
- R10, R11, R12, R13, R3, R5, R7, R9: PARTNO (none) -> RC0805JR-0710KL,YAGEO (VA),dk,311-10KARCT-ND,RES SMD 10K OH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
- R2, R4, R6, R8: PARTNO (none) -> MCR10EZPJ391,ROHM SEMICONDUCTOR (PASSIVE) (VA),DK,RHM390ARC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
- S1, S2, S3, S4: PARTNO (none) -> MJTP1230,Apem,dk,679-2428-ND,Tactile Switch SPST-NO Top Act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
- T1, T3: PARTNO (none) -> MMBT3904LT1G,on semiconductor,dk,MMBT3904LT1GOSCT-ND,TRANS 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
- U1: PARTNO (none) -> TSOP38238,VISHAY DALE (VA),dk,751-1227-ND,IC IR RCVR MOD 38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
- X1: PARTNO (none) -> 385646,AI-Thinker,dx.com,385646,ESP8266 Serial Wi-Fi Wirele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
