File: eCogs/eCog0_Blank.brd (EAGLE design)
At the start: 47.5 x 28 mm, 3 parts

Commit message: Updated to latest eCog Library
Parts:
- ECOG: value ECOG_GENERAL_ROWECOG_GENERAL_SMD -> ECOG_GENERAL_ROWSURFACEMOUNT
Changed lines of the file:
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@@
 </autorouter>
 <elements>
-<element name="ECOG" library="eCogs" package="ECOG_GENERAL_SMD" value="ECOG_GENERAL_ROWECOG_GENERAL_SMD" x="0" y="0" smashed="yes">
+<element name="ECOG" library="eCogs" package="ECOG_GENERAL_SMD" value="ECOG_GENERAL_ROWSURFACEMOUNT" x="0" y="0" smashed="yes">
 <attribute name="DIGIKEY" value="S1013EC-10-ND" x="0" y="0" size="1.778" layer="27" display="off"/>
 </element>
