File: eCogs/eCog100_ESP8266_Wifi.sch (EAGLE design)
At the start: 6 parts

Commit message: Updated to latest eCog Library
Parts:
- ECOG: value ECOG_GENERAL_ROWECOG_GENERAL_SMD -> ECOG_GENERAL_ROWSURFACEMOUNT; device eCogs:ECOG_GENERAL_ROWECOG_GENERAL_SMD -> eCogs:ECOG_GENERAL_ROWSURFACEMOUNT
Changed lines of the file:
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@@
 <part name="FRAME1" library="frames" deviceset="A3L-LOC" device=""/>
 <part name="GND2" library="GadgetFactory" deviceset="GND" device=""/>
-<part name="ECOG" library="eCogs" deviceset="ECOG_GENERAL_ROW" device="ECOG_GENERAL_SMD" value="ECOG_GENERAL_ROWECOG_GENERAL_SMD"/>
+<part name="ECOG" library="eCogs" deviceset="ECOG_GENERAL_ROW" device="SURFACEMOUNT" value="ECOG_GENERAL_ROWSURFACEMOUNT"/>
 <part name="X1" library="adafruit" deviceset="ESP-12" device="">
 <attribute name="ADAFRUIT" value="2491"/>
