File: eCogs/eCog101_I2C_TFT_.96.sch (EAGLE design)
At the start: 2 parts

Commit message: Updated to latest eCog Library
Parts:
- ECOG: value ECOG_BUSES_ROWECOG_BUSES_SMD -> ECOG_BUSES_ROWSURFACEMOUNT; device eCogs:ECOG_BUSES_ROWECOG_BUSES_SMD -> eCogs:ECOG_BUSES_ROWSURFACEMOUNT
Changed lines of the file:
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@@
 <part name="FRAME1" library="frames" deviceset="A3L-LOC" device=""/>
 <part name="GND2" library="GadgetFactory" deviceset="GND" device=""/>
-<part name="ECOG" library="eCogs" deviceset="ECOG_BUSES_ROW" device="ECOG_BUSES_SMD" value="ECOG_BUSES_ROWECOG_BUSES_SMD"/>
+<part name="ECOG" library="eCogs" deviceset="ECOG_BUSES_ROW" device="SURFACEMOUNT" value="ECOG_BUSES_ROWSURFACEMOUNT"/>
 <part name="JP1" library="pinhead" deviceset="PINHD-1X4" device="" value=".96 I2C OLED LCD">
 <attribute name="DEALEXTREME" value="419232"/>
