File: GadgetBox-Teensy/Gadget-Box-teensy.brd (EAGLE design)
At the start: 93.5 x 53.5 mm, 25 parts, among them U1 MCP73831T-2ACI/OT, U2 AP2112-3.3, U3 TEENSY_3.1_ALL_PINS

Commit message: Added BOM info
Parts:
- removed C1, C3: 10µF, microbuilder:0805-NO
- removed C4: 1uF, GadgetFactory:0603
- removed PWR: (no value), adafruit:USB-MINIB
- removed U2: AP2112-3.3, microbuilder:SOT23-5
- moved JP1 1.27 mm to (16.9, 52.1)
Connections:
- removed net 5V0: AH.5V@2, AL.5V@2, BH.5V@2, BL.5V@2, C1.1, CHG.A, D1.C, PSW1.1, PWR.VBUS, U1.4, U2.1, U3.VUSB
- removed net EN: PSW1.2, U2.3
- new net N$5: D1.C, PSW1.1
- new net VUSB: AH.5V@2, AL.5V@2, BH.5V@2, BL.5V@2, CHG.A, U1.4, U3.VUSB
- net 3V3: no longer C3.1, C4.2, U2.5
- net GND: no longer C1.2, C3.2, C4.1, PSW1.3, PWR.GND, U2.2
- net VIN: now also PSW1.2
Routing:
- net 5V0: track 226.5 -> 0.00 mm, vias 6 -> 0
- net VUSB: track 0.00 -> 219.3 mm, vias 0 -> 6
- net N$5: track 0.00 -> 111.4 mm, vias 0 -> 4
- net EN: track 72.6 -> 0.00 mm, vias 2 -> 0
- net VIN: track 0.00 -> 22.8 mm, vias 0 -> 1
- net GND: track 23.9 -> 10.4 mm, vias 6 -> 3
- net VBATTERY: track 43.7 -> 44.3 mm
Other:
- board text added: "Gadget Box - Teensy 3.2 Copyright 2016 Gadget Factory, LLC Version 1.1"
- board text removed: "Gadget Box - Teensy 3.2 Copyright 2016 Gadget Factory, LLC Version 1.0"
