File: hardware/GadgetBox-mini-pro/GadgetBox-Mini-Pro-Clone.sch (EAGLE design)
At the start: 27 parts, among them U1 MCP73831T-2ACI/OT, U2 AP2112-3.3

Commit message: Update License info
Other:
- note added: "This work is licensed under the Creative Commons Attribution-ShareAlike License."
- note added: "To view a copy of this license, visit http://creativecommons.org/ ; or, (b) send a letter to Creative Commons, 171 2nd Street, Suite 300, San Francisco, California, 94105, USA."
Changed lines of the file:
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@@
 <sheet>
 <plain>
+<text x="78.74" y="-5.08" size="1.778" layer="94">This work is licensed under the Creative Commons Attribution-ShareAlike License.</text>
+<text x="-2.54" y="-7.62" size="1.778" layer="94">To view a copy of this license, visit http://creativecommons.org/ ; or, (b) send a letter to Creative Commons, 171 2nd Street, Suite 300, San Francisco, California, 94105, USA.</text>
 </plain>
 <instances>
@@
 <wire x1="5.08" y1="71.12" x2="134.62" y2="71.12" width="0.1524" layer="94" style="shortdash"/>
 <text x="142.24" y="119.38" size="1.778" layer="94">Measure Battery (Populate R10 with 0 ohm jumper)</text>
+<text x="58.42" y="-5.08" size="1.778" layer="94">This work is licensed under the Creative Commons Attribution-ShareAlike License.</text>
+<text x="0" y="-7.62" size="1.778" layer="94">To view a copy of this license, visit http://creativecommons.org/ ; or, (b) send a letter to Creative Commons, 171 2nd Street, Suite 300, San Francisco, California, 94105, USA.</text>
 </plain>
 <instances>
